File: docs/kicad/examples/bridge.kicad_sch (KiCad schematic)
At the start: 8 parts

Commit message: fix: file watcher polling, cross-probe removal, guide updates
- Rewrite file watcher from QFileSystemWatcher to mtime polling (KiCad's
  rename-over atomic save silently breaks QFileSystemWatcher tracking)
- Replace "Simulate Now" with "Re-Watch" button (resumes watching after Stop)
- Remove cross-probe/back-annotation from menu and docs (KiCad's cross-probe
  channel is private Eeschema-PcbNew, not an external API)
- Document cross-probe as known limitation in user guide
- Rename back_annotate.kicad_sch to bjt_amplifier.kicad_sch
- Make all Help dialogs non-modal (show() instead of exec())
- Add Help > KiCad User Guide entry with pre-built HTML
- Persist traces across KiCad re-simulations
- Add raw_ok check in bridge.simulate() (ngspice can exit 0 without writing .raw)
- Fix _panel_grid -> panel_grid typo in cross-probe helper
- Initialize all KiCad-related instance attributes

Co-Authored-By: Claude Opus 4.7 <noreply@anthropic.com>
Parts:
- C1: value 47u -> 47uF
Other:
- note added: ".tran 100u 50m"
Changed lines of the file:
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@@
 	(generator_version "9.0")
 	(paper "A4")
+	(text ".tran 100u 50m"
+		(exclude_from_sim no)
+		(at 98.298 134.62 0)
+		(effects
+			(font
+				(size 1.27 1.27)
+			)
+		)
+	)
 	(text ".model D1N4148 D(Is=2.55e-9 N=1.75 Rs=42e-3 Cj0=42.4e-12 Vj=0.75 M=0.333 Fc=0.5 Tt=4.32e-6 Bv=800 Ibv=80e-6 Af=1 Kf=0)"
 		(exclude_from_sim no)
@@
 			)
 		)
-		(property "Value" "47u"
+		(property "Value" "47uF"
 			(at 99.06 93.3449 0)
 			(effects
